Commit message: feat(sensor): integrate 2D LiDAR and configure ROS-GZ bridge
- Add lidar_link and gpu_lidar plugin to my_robot.urdf
- Map /scan topic in bridge_params.yaml (GZ -> ROS)
- Update sim_launch.py to use 'shapes.sdf' for obstacle testing
- Add static_transform_publisher to fix Gazebo frame lumping issue

File: src/my_robot_controller/urdf/my_robot.urdf (robot description, URDF)
Before this commit: robot my_robot, 5 links, 4 joints
Links:
- added link lidar_link, mass 0.1; collision cylinder length=0.04 radius=0.05; visual cylinder length=0.04 radius=0.05
Joints:
- added joint lidar_joint: type fixed, parent base_link, child lidar_link, origin xyz=0 0 0.12 rpy=0 0 0

Commit message: Refactor: Switch to Bumperbot URDF and Fix Physics
Replaced custom robot model with Bumperbot URDF. Optimized wheel friction and torque limits to fix odometry drift. Added generated SLAM map (my_map).

File: src/my_robot_controller/urdf/my_robot.urdf (robot description, URDF)
Before this commit: robot my_robot, 6 links, 5 joints
Links:
- removed link caster_front
- removed link caster_rear
- removed link left_wheel
- removed link lidar_link
- removed link right_wheel
- added link base_footprint
- added link caster_front_link, mass 0.001; collision sphere radius=0.015; visual sphere radius=0.015
- added link caster_rear_link, mass 0.001; collision sphere radius=0.015; visual sphere radius=0.015
- added link laser_link, mass 0.07; collision cylinder length=0.04 radius=0.04; visual cylinder length=0.04 radius=0.04
- added link wheel_left_link, mass 0.053; collision cylinder length=0.02 radius=0.033; visual cylinder length=0.02 radius=0.033
- added link wheel_right_link, mass 0.053; collision cylinder length=0.02 radius=0.033; visual cylinder length=0.02 radius=0.033
- link base_link: mass 10.0 -> 0.8257; geometry collision box size=0.3 0.3 0.15; visual box size=0.3 0.3 0.15
Joints:
- removed joint base_to_left_wheel
- removed joint base_to_right_wheel
- removed joint lidar_joint
- added joint base_joint: type fixed, parent base_footprint, child base_link, origin xyz=0 0 0.033 rpy=0 0 0
- added joint laser_joint: type fixed, parent base_link, child laser_link, origin xyz=0 0 0.12 rpy=0 0 0
- added joint wheel_left_joint: type continuous, parent base_link, child wheel_left_link, origin xyz=0 0.12 0 rpy=0 0 0, axis 0 1 0
- added joint wheel_right_joint: type continuous, parent base_link, child wheel_right_link, origin xyz=0 -0.12 0 rpy=0 0 0, axis 0 1 0
- joint caster_front_joint: child caster_front -> caster_front_link; origin xyz=0.25 0 -0.15 -> xyz=0.12 0 -0.018 rpy=0 0 0
- joint caster_rear_joint: child caster_rear -> caster_rear_link; origin xyz=-0.25 0 -0.15 -> xyz=-0.12 0 -0.018 rpy=0 0 0

Commit message: feat: map changed to more complex map

File: src/my_robot_controller/urdf/my_robot.urdf (robot description, URDF)
Before this commit: robot bumperbot, 7 links, 6 joints
Links:
- link caster_front_link: mass 0.001 -> 0.05
- link caster_rear_link: mass 0.001 -> 0.05
- link wheel_left_link: mass 0.053 -> 0.2
- link wheel_right_link: mass 0.053 -> 0.2
Joints:
- joint caster_front_joint: type fixed -> continuous
- joint caster_rear_joint: type fixed -> continuous

Commit message: add: Added camera to my_robot_urdf

File: src/my_robot_controller/urdf/my_robot.urdf (robot description, URDF)
Before this commit: robot bumperbot, 7 links, 6 joints
Links:
- added link camera_link, mass 0.05; collision box size=0.04 0.04 0.04; visual box size=0.04 0.04 0.04
Joints:
- added joint camera_joint: type fixed, parent base_link, child camera_link, origin xyz=0.10 0.06 0.18 rpy=0 0 0

Commit message: refactor(urdf): switch kinematics from Diff Drive to Ackermann steering
- Replace DiffDrive plugin with AckermannSteering in URDF
- Configure steering and traction joints with correct limits
- Update ROS-GZ bridge topics (YAML/config) to match new Ackermann nodes

File: src/my_robot_controller/urdf/my_robot.urdf (robot description, URDF)
Before this commit: robot bumperbot, 8 links, 7 joints
Links:
- removed link caster_front_link
- removed link caster_rear_link
- removed link wheel_left_link
- removed link wheel_right_link
- added link front_left_steering_link, mass 0.01
- added link front_left_wheel_link, mass 0.2; collision cylinder length=0.02 radius=0.033; visual cylinder length=0.02 radius=0.033
- added link front_right_steering_link, mass 0.01
- added link front_right_wheel_link, mass 0.2; collision cylinder length=0.02 radius=0.033; visual cylinder length=0.02 radius=0.033
- added link rear_left_wheel_link, mass 0.2; collision cylinder length=0.02 radius=0.033; visual cylinder length=0.02 radius=0.033
- added link rear_right_wheel_link, mass 0.2; collision cylinder length=0.02 radius=0.033; visual cylinder length=0.02 radius=0.033
- link base_link: mass 0.8257 -> 2.0; geometry collision box size=0.4 0.20 0.1; visual box size=0.4 0.20 0.1
Joints:
- removed joint caster_front_joint
- removed joint caster_rear_joint
- removed joint wheel_left_joint
- removed joint wheel_right_joint
- added joint front_left_steering_joint: type revolute, parent base_link, child front_left_steering_link, origin xyz=0.12 0.14 0 rpy=0 0 0, axis 0 0 1, limit lower=-0.6 upper=0.6 effort=10 velocity=10
- added joint front_left_wheel_joint: type continuous, parent front_left_steering_link, child front_left_wheel_link, origin xyz=0 0 0 rpy=0 0 0, axis 0 1 0
- added joint front_right_steering_joint: type revolute, parent base_link, child front_right_steering_link, origin xyz=0.12 -0.14 0 rpy=0 0 0, axis 0 0 1, limit lower=-0.6 upper=0.6 effort=10 velocity=10
- added joint front_right_wheel_joint: type continuous, parent front_right_steering_link, child front_right_wheel_link, origin xyz=0 0 0 rpy=0 0 0, axis 0 1 0
- added joint rear_left_wheel_joint: type continuous, parent base_link, child rear_left_wheel_link, origin xyz=-0.12 0.14 0 rpy=0 0 0, axis 0 1 0
- added joint rear_right_wheel_joint: type continuous, parent base_link, child rear_right_wheel_link, origin xyz=-0.12 -0.14 0 rpy=0 0 0, axis 0 1 0
- joint camera_joint: origin xyz=0.10 0.06 0.18 rpy=0 0 0 -> xyz=0.19 0 0.15 rpy=0 0 0
- joint laser_joint: origin xyz=0 0 0.12 rpy=0 0 0 -> xyz=0 0 0.14 rpy=0 0 0

Commit message: refactor(sim): switch to EKF-based TF, tune URDF physics and planner params
- Localization: Designate robot_localization (EKF) as the sole provider of the 'odom' -> 'base_footprint' TF.

- URDF: Increase steering link mass and add wheel friction/stiffness (kp/kd) to fix simulation jitter.

- Nav2: Add change_penalty parameter

File: src/my_robot_controller/urdf/my_robot.urdf (robot description, URDF)
Before this commit: robot bumperbot, 10 links, 9 joints
Links:
- link front_left_steering_link: mass 0.01 -> 0.1
- link front_right_steering_link: mass 0.01 -> 0.1

Commit message: feat: integrate IMU, fix odom drift and update nav2 params
- Added IMU sensor to URDF and configured EKF fusion.
- Fixed odometry drift and sideslip issues.
- Increased vehicle mass in URDF for better physics simulation.
- Tuned Nav2 parameters (planner/controller) for smoother navigation.

File: src/my_robot_controller/urdf/my_robot.urdf (robot description, URDF)
Before this commit: robot bumperbot, 10 links, 9 joints
Links:
- added link imu_link, mass 0.01; collision box size=0.02 0.02 0.02; visual box size=0.02 0.02 0.02
- link base_link: mass 2.0 -> 10.0
Joints:
- added joint imu_joint: type fixed, parent base_link, child imu_link, origin xyz=0 0 0.1 rpy=0 0 0

Commit message: feat(sim): add textured robotaksi map and configure rendering
- Integrated RobotaksiMap as a .dae model for texture compatibility in Gazebo.
- Sanitized texture file names and fixed path encodings within the collada file.
- Zeroed map pose to align correctly with the invisible ground collision plane.
- Enabled proper camera image rendering in headless mode via Xvfb.

File: src/my_robot_controller/urdf/my_robot.urdf (robot description, URDF)
Before this commit: robot bumperbot, 11 links, 10 joints
Links:
- added link camera_gta_link, mass 0.01; visual box size=0.01 0.01 0.01
Joints:
- added joint camera_gta_joint: type fixed, parent base_link, child camera_gta_link, origin xyz=-0.8 0 0.8 rpy=0 0.5 0

Commit message: feat: kamera GTA view düzeltildi, dashboard kamera sekmesi eklendi

File: src/my_robot_controller/urdf/my_robot.urdf (robot description, URDF)
Before this commit: robot bumperbot, 12 links, 11 joints
Joints:
- joint camera_gta_joint: origin xyz=-0.8 0 0.8 rpy=0 0.5 0 -> xyz=0 0 8.0 rpy=0 1.5707 0

Commit message: feat: scale up robot to match Robotaksi competition dimensions
- URDF: vehicle body 0.4x0.2m -> 2.0x1.2m (competition min 200x120cm)
- URDF: wheel radius 3.3cm -> 16.5cm, wheelbase 0.24 -> 1.2m
- URDF: camera pitch adjusted for lane detection (rpy 0 0.3 0)
- nav2: footprint updated [0.22,0.12] -> [1.0,0.6]
- nav2: min_turning_radius 1.0 -> 2.5m (wheelbase=1.2m)
- nav2: costmap 3x3 -> 8x8, inflation_radius 0.55 -> 1.2m
- nav2: lidar range 3.5m -> 10m, vx_max 1.0 -> 2.0

File: src/my_robot_controller/urdf/my_robot.urdf (robot description, URDF)
Before this commit: robot bumperbot, 12 links, 11 joints
Links:
- link base_link: mass 10.0 -> 500.0; geometry collision box size=2.0 1.2 0.4; visual box size=2.0 1.2 0.4
- link camera_gta_link: mass 0.01 -> 0.05; geometry visual box size=0.05 0.05 0.05
- link camera_link: mass 0.05 -> 0.2; geometry collision box size=0.1 0.1 0.1; visual box size=0.1 0.1 0.1
- link front_left_steering_link: mass 0.1 -> 1.0
- link front_left_wheel_link: mass 0.2 -> 5.0; geometry collision cylinder length=0.1 radius=0.165; visual cylinder length=0.1 radius=0.165
- link front_right_steering_link: mass 0.1 -> 1.0
- link front_right_wheel_link: mass 0.2 -> 5.0; geometry collision cylinder length=0.1 radius=0.165; visual cylinder length=0.1 radius=0.165
- link imu_link: mass 0.01 -> 0.05; geometry collision box size=0.05 0.05 0.05; visual box size=0.05 0.05 0.05
- link laser_link: mass 0.07 -> 0.5; geometry collision cylinder length=0.1 radius=0.1; visual cylinder length=0.1 radius=0.1
- link rear_left_wheel_link: mass 0.2 -> 5.0; geometry collision cylinder length=0.1 radius=0.165; visual cylinder length=0.1 radius=0.165
- link rear_right_wheel_link: mass 0.2 -> 5.0; geometry collision cylinder length=0.1 radius=0.165; visual cylinder length=0.1 radius=0.165
Joints:
- joint base_joint: origin xyz=0 0 0.033 rpy=0 0 0 -> xyz=0 0 0.165 rpy=0 0 0
- joint camera_gta_joint: origin xyz=0 0 8.0 rpy=0 1.5707 0 -> xyz=0 0 15.0 rpy=0 1.5707 0
- joint camera_joint: origin xyz=0.19 0 0.15 rpy=0 0 0 -> xyz=0.95 0 0.5 rpy=0 0.3 0
- joint front_left_steering_joint: limit lower=-0.6 upper=0.6 effort=10 velocity=10 -> lower=-0.6 upper=0.6 effort=100 velocity=10; origin xyz=0.12 0.14 0 rpy=0 0 0 -> xyz=0.6 0.65 0 rpy=0 0 0
- joint front_right_steering_joint: limit lower=-0.6 upper=0.6 effort=10 velocity=10 -> lower=-0.6 upper=0.6 effort=100 velocity=10; origin xyz=0.12 -0.14 0 rpy=0 0 0 -> xyz=0.6 -0.65 0 rpy=0 0 0
- joint imu_joint: origin xyz=0 0 0.1 rpy=0 0 0 -> xyz=0 0 0.4 rpy=0 0 0
- joint laser_joint: origin xyz=0 0 0.14 rpy=0 0 0 -> xyz=0 0 0.6 rpy=0 0 0
- joint rear_left_wheel_joint: origin xyz=-0.12 0.14 0 rpy=0 0 0 -> xyz=-0.6 0.65 0 rpy=0 0 0
- joint rear_right_wheel_joint: origin xyz=-0.12 -0.14 0 rpy=0 0 0 -> xyz=-0.6 -0.65 0 rpy=0 0 0

Commit message: lane

File: src/my_robot_controller/urdf/my_robot.urdf (robot description, URDF)
Before this commit: robot bumperbot, 12 links, 11 joints
Joints:
- joint camera_joint: origin xyz=0.95 0 0.5 rpy=0 0.3 0 -> xyz=0.95 0 1.2 rpy=0 0.35 0
